File: ReBlast.kicad_pcb (KiCad board)
At the start: 2 copper layers, 50.7 x 63.8 mm, 21 parts, among them J1 MOS_8580_Socket, U1 74HC20, U2 74LS139, U3 ZN428E-8, U4 TLC272, U5 MOS_8580

Commit message: Checkpoint!
Parts:
- U2: value 74LS139 -> 74HC139
Connections:
- J1 pad 10: Net-(J1-Pad10) -> /a1
- J1 pad 11: Net-(J1-Pad11) -> /a2
- J1 pad 12: Net-(J1-Pad12) -> /a3
- J1 pad 13: Net-(J1-Pad13) -> /a4
- J1 pad 9: Net-(J1-Pad9) -> /a0
- U1 pad 1: Net-(U1-Pad1) -> /a3
- U1 pad 14: Net-(U1-Pad14) -> +5V
- U1 pad 7: Net-(U1-Pad7) -> GNDD
- U2 pad 16: Net-(U2-Pad16) -> +5V
- U2 pad 3: Net-(U2-Pad3) -> Net-(U1-Pad6)
- U2 pad 8: Net-(U2-Pad8) -> GNDD
- U5 pad 10: Net-(U5-Pad10) -> /a1
- U5 pad 11: Net-(U5-Pad11) -> /a2
- U5 pad 12: Net-(U5-Pad12) -> /a3
- U5 pad 13: Net-(U5-Pad13) -> /a4
- U5 pad 9: Net-(U5-Pad9) -> /a0
Routing:
- net /a3: track 0.00 -> 19.7 mm
- net +5V: track 0.00 -> 13.3 mm
- net Net-(U1-Pad6): track 0.00 -> 12.8 mm
- net /a4: track 0.00 -> 11.0 mm
Other:
- board size 50.7 x 63.8 mm -> 50.7 x 64.9 mm
- net class Default: via_dia 0.8 -> 0.6
- net class Power added: clearance 0.2, trace_width 0.5, via_dia 0.8, via_drill 0.6

Commit message: Suppositions in progress...
Parts:
- added C7: CP1, Capacitor_THT:CP_Radial_D5.0mm_P2.00mm, F.Cu at (150.6, 80.6)
- C2: footprint Capacitor_THT:CP_Radial_D5.0mm_P2.00mm -> Capacitor_THT:C_Disc_D7.0mm_W2.5mm_P5.00mm
- moved C2 16.9 mm to (167.5, 80.5), turned to 0 degrees
Connections:
- net Net-(U1-Pad6) renamed /~digiaddr
- net Net-(U2-Pad10) renamed /~cs_adc_w
- net Net-(U2-Pad11) renamed /~cs_dac_r
- net Net-(U2-Pad12) renamed /~cs_dac_w
- net Net-(U2-Pad9) renamed /~cs_adc_r
- D3 pad 1: Net-(D3-Pad1) -> GNDD
- D3 pad 2: Net-(D3-Pad2) -> Net-(D2-Pad1)
- J1 pad 8: /~cs -> /~cs_in
- U1 pad 2: Net-(U1-Pad2) -> /a2
- U1 pad 4: Net-(U1-Pad4) -> /a1
- U1 pad 5: Net-(U1-Pad5) -> /a4
- U2 pad 1: Net-(U2-Pad1) -> /~cs_in
- U2 pad 13: Net-(U2-Pad13) -> /a0
- U2 pad 14: Net-(U2-Pad14) -> /r_~w
- U2 pad 15: Net-(U2-Pad15) -> /~cs_dac_adc
- U2 pad 2: Net-(U2-Pad2) -> GNDD
- U2 pad 4: Net-(U2-Pad4) -> /~cs_dac_adc
- U2 pad 6: Net-(U2-Pad6) -> /~cs_sid
- U5 pad 8: /~cs -> /~cs_sid

Commit message: Back side is 99% done. Top side is full of doubts...
Parts:
- added U6: ADC0804, Package_DIP:DIP-20_W7.62mm, F.Cu at (162.1, 112.3)
- C1: footprint Capacitor_THT:C_Disc_D7.0mm_W2.5mm_P5.00mm -> Capacitor_THT:C_Disc_D5.0mm_W2.5mm_P2.50mm
- C2: value C_TANTALUM -> 4.7u; footprint Capacitor_THT:C_Disc_D7.0mm_W2.5mm_P5.00mm -> Capacitor_THT:C_Disc_D5.0mm_W2.5mm_P2.50mm
- C4: value CP1 -> C
- C6: footprint Capacitor_THT:CP_Radial_D8.0mm_P5.00mm -> Capacitor_THT:CP_Radial_D6.3mm_P2.50mm
- C7: value CP1 -> 6.8u
- D1: value 1n4148 -> 2.5V ZENER
- J1: footprint ReBlast:DIP-28_Socket_LongPads -> Package_DIP:DIP-28_W15.24mm
- R2: value 4.7k -> 47k
- R3: footprint Resistor_THT:R_Axial_DIN0414_L11.9mm_D4.5mm_P15.24mm_Horizontal -> Resistor_THT:R_Axial_DIN0207_L6.3mm_D2.5mm_P7.62mm_Horizontal
- R4: value 10K or 120 -> 10K
- U3: footprint Package_DIP:DIP-16_W7.62mm_Socket_LongPads -> Package_DIP:DIP-16_W7.62mm_Socket
- U4: footprint Package_DIP:DIP-8_W7.62mm_Socket_LongPads -> Package_DIP:DIP-8_W7.62mm_Socket
- U5: footprint Package_DIP:DIP-28_W15.24mm_Socket_LongPads -> Package_DIP:DIP-28_W15.24mm_Socket
- moved R4 7.78 mm to (136.1, 79.1)
- moved R1 7.68 mm to (174.8, 84.3), turned to 90 degrees
- moved C5 7.13 mm to (137.3, 95.7), turned to 270 degrees
- moved D2 5.20 mm to (150.6, 86.9), turned to 180 degrees
- moved C2 5.00 mm to (172.5, 80.5), turned to 180 degrees
- moved C1 4.18 mm to (139.2, 79.1), turned to 0 degrees
- moved R3 4.07 mm to (139.2, 83.0)
- moved C4 2.98 mm to (146.8, 91.3)
- moved J1 1.27 mm to (129.0, 122.4)
- moved C3 1.21 mm to (149.4, 91.3), turned to 0 degrees
- moved C6 1.20 mm to (144.3, 81.8), turned to 270 degrees
- moved D3 0.58 mm to (148.1, 84.3), turned to 0 degrees
- moved C7 0.40 mm to (150.7, 80.3)
- moved D1 0.06 mm to (172.5, 84.3)
- moved U4 0.06 mm to (162.1, 91.9)
Connections:
- net /~cs_adc_r renamed Net-(U2-Pad9)
- net /~cs_adc_w renamed Net-(U2-Pad10)
- net /~cs_dac_w renamed Net-(U2-Pad12)
- net Net-(C3-Pad1) renamed /vref
- C2 pad 1: Net-(C2-Pad1) -> Net-(C1-Pad2)
- C4 pad 1: Net-(C4-Pad1) -> /dac_output
- C4 pad 2: Net-(C4-Pad2) -> /audio_in
- C5 pad 2: Net-(C5-Pad2) -> /audio_jack
- C6 pad 1: Net-(C6-Pad1) -> Net-(C1-Pad1)
- C6 pad 2: Net-(C6-Pad2) -> GNDA
- C7 pad 2: Net-(C7-Pad2) -> Net-(C1-Pad2)
- D1 pad 1: Net-(D1-Pad1) -> Net-(C1-Pad2)
- D1 pad 2: Net-(D1-Pad2) -> Net-(C2-Pad2)
- D3 pad 1: GNDD -> Net-(C5-Pad1)
- D3 pad 2: Net-(D2-Pad1) -> Net-(D3-Pad2)
- J1 pad 14: GNDD -> GNDA
- J1 pad 26: Net-(J1-Pad26) -> /audio_jack
- R1 pad 1: Net-(R1-Pad1) -> Net-(C1-Pad1)
- R2 pad 2: Net-(R2-Pad2) -> Net-(C2-Pad2)
- R3 pad 1: Net-(R3-Pad1) -> Net-(C1-Pad1)
- R4 pad 1: Net-(R4-Pad1) -> Net-(D3-Pad2)
- R4 pad 2: Net-(R4-Pad2) -> Net-(C5-Pad1)
- RV1 pad 1: Net-(RV1-Pad1) -> Net-(R1-Pad2)
- RV1 pad 3: Net-(RV1-Pad3) -> Net-(C1-Pad2)
- U1 pad 10: Net-(U1-Pad10) -> +5V
- U1 pad 12: Net-(U1-Pad12) -> +5V
- U1 pad 13: Net-(U1-Pad13) -> +5V
- U1 pad 2: /a2 -> /a4
- U1 pad 4: /a1 -> /a2
- U1 pad 5: /a4 -> /a1
- U1 pad 7: GNDD -> GNDA
- U2 pad 11: /~cs_dac_r -> /~cs_sid
- U2 pad 13: /a0 -> GNDA
- U2 pad 14: /r_~w -> /~digiaddr
- U2 pad 15: /~cs_dac_adc -> /~cs_in
- U2 pad 2: GNDD -> /a0
- U2 pad 4: /~cs_dac_adc -> /~cs_dac
- U2 pad 5: Net-(U2-Pad5) -> /~cs_adc
- U2 pad 6: /~cs_sid -> Net-(U2-Pad6)
- U2 pad 8: GNDD -> GNDA
- U3 pad 1: /d6 -> /d1
- U3 pad 11: /d0 -> /d7
- U3 pad 12: /d1 -> /d6
- U3 pad 13: /d2 -> /d5
- U3 pad 14: /d3 -> /d4
- U3 pad 15: /d4 -> /d3
- U3 pad 16: /d5 -> /d2
- U3 pad 2: /d7 -> /d0
- U3 pad 4: Net-(U3-Pad4) -> /~cs_dac
- U3 pad 5: Net-(U3-Pad5) -> /dac_output
- U3 pad 9: GNDD -> GNDA
- U4 pad 1: Net-(U4-Pad1) -> Net-(D2-Pad2)
- U4 pad 2: Net-(U4-Pad2) -> Net-(D2-Pad1)
- U4 pad 4: Net-(U4-Pad4) -> GNDA
- U4 pad 5: Net-(U4-Pad5) -> Net-(C7-Pad1)
- U4 pad 6: Net-(U4-Pad6) -> Net-(D3-Pad2)
- U4 pad 8: Net-(U4-Pad8) -> +5V
- U5 pad 14: GNDD -> GNDA
Routing:
- net GNDA: track 0.00 -> 140.8 mm
- net (no net): track 0.00 -> 137.4 mm, vias 0 -> 1
- net +5V: track 13.3 -> 80.1 mm
- net /~cs_sid: track 0.00 -> 55.6 mm
- net /~cs_in: track 0.00 -> 54.9 mm
- net Net-(C1-Pad1): track 0.00 -> 51.3 mm
- net /a0: track 0.00 -> 47.5 mm
- net Net-(C1-Pad2): track 0.00 -> 43.1 mm
- net /audio_in: track 0.00 -> 37.7 mm
- net /d0: track 0.00 -> 32.9 mm
- net Net-(C2-Pad2): track 0.00 -> 30.9 mm
- net /a1: track 0.00 -> 30.9 mm
- net /d1: track 0.00 -> 27.3 mm
- net /~cs_dac: track 0.00 -> 27.3 mm, vias 0 -> 1
- net /a2: track 0.00 -> 26.0 mm
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- added copper zone on B.Cu, net GNDD
- added copper zone on F.Cu, net GNDD
Other:
- outline, holes or cut-outs redrawn

Commit message: Power circuit almost makes sense
Parts:
- removed R3: 100R 1/2W, Resistor_THT:R_Axial_DIN0207_L6.3mm_D2.5mm_P7.62mm_Horizontal
- added L1: 100, Inductor_THT:L_Axial_L6.6mm_D2.7mm_P10.16mm_Horizontal_Vishay_IM-2, F.Cu at (139.2, 93.1)
- R2: value 47k -> 4.7k
Connections:
- C1 pad 1: Net-(C1-Pad1) -> +5V
- C6 pad 1: Net-(C1-Pad1) -> +5V
- D3 pad 1: Net-(C5-Pad1) -> Net-(D3-Pad1)
- J1 pad 25: +5V -> VCC
- R1 pad 1: Net-(C1-Pad1) -> +5V
- U5 pad 25: +5V -> VCC
Routing:
- net +5V: track 80.1 -> 150.9 mm
- net Net-(C1-Pad1): track 51.3 -> 0.00 mm
- net VCC: track 0.00 -> 17.7 mm
- net Net-(R3-Pad2): track 17.5 -> 0.00 mm
- net /audio_in: track 37.7 -> 35.1 mm
- net Net-(D2-Pad1): track 12.5 -> 14.6 mm
- net Net-(U4-Pad7): track 2.22 -> 4.10 mm

Commit message: Nothing makes sense
Parts:
- removed D2, D3: 1N5817, Diode_THT:D_DO-41_SOD81_P2.54mm_Vertical_AnodeUp
- added R3: R, Resistor_THT:R_Axial_DIN0207_L6.3mm_D2.5mm_P2.54mm_Vertical, F.Cu at (150.6, 85.5)
- added R6: R, Resistor_THT:R_Axial_DIN0207_L6.3mm_D2.5mm_P2.54mm_Vertical, F.Cu at (148.1, 88.1)
- C2: value 4.7u -> CERAMIC
- C4: value C -> 1u
- C6: value CP1 -> 1u
- C7: value 6.8u -> 1u
- moved C2 2.50 mm to (170.0, 80.5), turned to 0 degrees
- moved C6 0.06 mm to (144.3, 81.8)
Connections:
- C1 pad 2: Net-(C1-Pad2) -> GNDA
- C2 pad 1: Net-(C1-Pad2) -> Net-(C2-Pad1)
- C2 pad 2: Net-(C2-Pad2) -> GNDA
- C7 pad 2: Net-(C1-Pad2) -> GNDA
- D1 pad 1: Net-(C1-Pad2) -> GNDA
- D1 pad 2: Net-(C2-Pad2) -> Net-(C2-Pad1)
- R2 pad 1: Net-(R2-Pad1) -> Net-(R1-Pad2)
- R2 pad 2: Net-(C2-Pad2) -> Net-(C2-Pad1)
- RV1 pad 3: Net-(C1-Pad2) -> GNDA
Routing:
- net GNDA: track 140.8 -> 196.5 mm
- net Net-(C1-Pad2): track 43.1 -> 0.00 mm
- net Net-(C2-Pad2): track 30.9 -> 0.00 mm
- net Net-(C2-Pad1): track 0.00 -> 30.9 mm
- net Net-(R1-Pad2): track 11.0 -> 22.5 mm
- net (no net): track 137.4 -> 130.1 mm
- net Net-(R6-Pad2): track 14.6 -> 12.0 mm
- net Net-(R6-Pad1): track 17.0 -> 15.5 mm
- net Net-(R3-Pad1): track 25.5 -> 24.9 mm

Commit message: Done?
Parts:
- C3: value 1u -> 4.7u
- C6: value 1u -> 47u
- R3, R6: value R -> 330k
- R4: value 10K -> 100k
Connections:
- C7 pad 1: Net-(C7-Pad1) -> Net-(C2-Pad1)
- R2 pad 1: Net-(R1-Pad2) -> +5V
- R3 pad 2: GNDA -> /adc_in
- R6 pad 1: Net-(R6-Pad1) -> /adc_vref_half
- U1 pad 10: +5V -> VCC
- U1 pad 12: +5V -> VCC
- U1 pad 13: +5V -> VCC
- U1 pad 14: +5V -> VCC
- U1 pad 8: Net-(U1-Pad8) -> /~read
- U1 pad 9: Net-(U1-Pad9) -> /r_~w
- U2 pad 16: +5V -> VCC
- U4 pad 1: Net-(R6-Pad1) -> /adc_vref_half
- U4 pad 3: Net-(U4-Pad3) -> Net-(RV1-Pad2)
- U4 pad 5: Net-(C7-Pad1) -> Net-(C2-Pad1)
- U4 pad 7: Net-(U4-Pad7) -> /adc_in
- U6 pad 2: Net-(U6-Pad2) -> /~read
- U6 pad 4: Net-(U6-Pad4) -> /phi2
- U6 pad 6: Net-(U6-Pad6) -> /adc_in
- U6 pad 7: Net-(U6-Pad7) -> GNDA
- U6 pad 8: Net-(U6-Pad8) -> GNDA
- U6 pad 9: Net-(U6-Pad9) -> /adc_vref_half
Routing:
- net (no net): track 130.1 -> 0.00 mm, vias 1 -> 0
- net VCC: track 17.7 -> 82.4 mm
- net /adc_vref_half: track 0.00 -> 54.2 mm
- net /r_~w: track 9.84 -> 54.4 mm
- net /adc_in: track 0.00 -> 35.5 mm
- net +5V: track 150.6 -> 181.9 mm, vias 0 -> 1
- net /phi2: track 2.54 -> 22.0 mm
- net GNDA: track 196.5 -> 215.8 mm
- net Net-(RV1-Pad2): track 0.00 -> 17.2 mm
- net Net-(R6-Pad1): track 15.5 -> 0.00 mm
- net Net-(U6-Pad4): track 12.4 -> 0.00 mm
- net Net-(C2-Pad1): track 30.9 -> 42.8 mm
- net Net-(R1-Pad2): track 22.5 -> 11.0 mm
- net /~read: track 0.00 -> 9.83 mm
- net Net-(U1-Pad9): track 7.18 -> 0.00 mm
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
Commit message: Try to come up with some values for caps
Parts:
- C1, C2: value CERAMIC -> 100n
Changed lines of the file:
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@@
   (general
     (thickness 1.6)
-    (drawings 14)
+    (drawings 10)
     (tracks 391)
     (zones 0)
@@
   (layers
     (0 F.Cu signal)
-    (31 B.Cu signal)
+    (31 B.Cu signal hide)
     (36 B.SilkS user)
     (37 F.SilkS user)
@@
     (descr "16-lead though-hole mounted DIP package, row spacing 7.62 mm (300 mils), Socket")
     (tags "THT DIP DIL PDIP 2.54mm 7.62mm 300mil Socket")
-    (fp_text reference U3 (at 3.81 -2.33 90) (layer F.SilkS)
-      (effects (font (size 1 1) (thickness 0.15)))
-    )
-    (fp_text value ZN428E-8 (at 3.81 20.11 90) (layer F.Fab)
+    (fp_text reference U3 (at 3.7325 -2.667 180) (layer F.SilkS)
+      (effects (font (size 1 1) (thickness 0.15)))
+    )
+    (fp_text value ZN428E-8 (at 3.7325 8.9 180) (layer F.SilkS)
       (effects (font (size 1 1) (thickness 0.15)))
     )
@@
     (descr "CP, Radial series, Radial, pin pitch=2.00mm, , diameter=5mm, Electrolytic Capacitor")
     (tags "CP Radial series Radial pin pitch 2.00mm  diameter 5mm Electrolytic Capacitor")
-    (fp_text reference C3 (at 4.064 -2.032) (layer F.SilkS)
-      (effects (font (size 1 1) (thickness 0.15)))
+    (fp_text reference C3 (at 2.921 -2.921) (layer F.SilkS)
+      (effects (font (size 0.8 0.8) (thickness 0.12)))
     )
     (fp_text value 4.7u (at 1 3.75) (layer F.Fab)
@@
     (descr "CP, Radial series, Radial, pin pitch=2.00mm, , diameter=5mm, Electrolytic Capacitor")
     (tags "CP Radial series Radial pin pitch 2.00mm  diameter 5mm Electrolytic Capacitor")
-    (fp_text reference C5 (at -2.477999 0.635 180) (layer F.SilkS)
+    (fp_text reference C5 (at 4.634001 0 180) (layer F.SilkS)
       (effects (font (size 1 1) (thickness 0.15)))
     )
@@
     (descr "Resistor, Axial_DIN0204 series, Axial, Horizontal, pin pitch=7.62mm, 0.167W, length*diameter=3.6*1.6mm^2, http://cdn-reichelt.de/documents/datenblatt/B400/1_4W%23YAG.pdf")
     (tags "Resistor Axial_DIN0204 series Axial Horizontal pin pitch 7.62mm 0.167W length 3.6mm diameter 1.6mm")
-    (fp_text reference R1 (at -1.8415 0.0635 180) (layer F.SilkS)
+    (fp_text reference R1 (at 9.271 0 180) (layer F.SilkS)
       (effects (font (size 1 1) (thickness 0.15)))
     )
@@
     (descr "14-lead though-hole mounted DIP package, row spacing 7.62 mm (300 mils), Socket, LongPads")
     (tags "THT DIP DIL PDIP 2.54mm 7.62mm 300mil Socket LongPads")
-    (fp_text reference U1 (at 10.2235 15.1765) (layer F.SilkS)
+    (fp_text reference U1 (at 3.8 -2.286) (layer F.SilkS)
       (effects (font (size 1 1) (thickness 0.15)))
     )
@@
     (descr "16-lead though-hole mounted DIP package, row spacing 7.62 mm (300 mils), Socket, LongPads")
     (tags "THT DIP DIL PDIP 2.54mm 7.62mm 300mil Socket LongPads")
-    (fp_text reference U2 (at 10.2235 0.064999) (layer F.SilkS)
+    (fp_text reference U2 (at 10.414 1.27) (layer F.SilkS)
       (effects (font (size 1 1) (thickness 0.15)))
     )
@@
     (descr "CP, Radial series, Radial, pin pitch=2.00mm, , diameter=5mm, Electrolytic Capacitor")
     (tags "CP Radial series Radial pin pitch 2.00mm  diameter 5mm Electrolytic Capacitor")
-    (fp_text reference C7 (at -1.5875 2.794) (layer F.SilkS)
+    (fp_text reference C7 (at -1.9685 2.286) (layer F.SilkS)
       (effects (font (size 1 1) (thickness 0.15)))
     )
@@
     (descr "8-lead though-hole mounted DIP package, row spacing 7.62 mm (300 mils), Socket")
     (tags "THT DIP DIL PDIP 2.54mm 7.62mm 300mil Socket")
-    (fp_text reference U4 (at 3.81 -2.33) (layer F.SilkS)
-      (effects (font (size 1 1) (thickness 0.15)))
-    )
-    (fp_text value TLC272 (at 3.81 9.95) (layer F.Fab)
+    (fp_text reference U4 (at -0.889 -2.54) (layer F.SilkS)
+      (effects (font (size 1 1) (thickness 0.15)))
+    )
+    (fp_text value TLC272 (at 3.8675 3.799999 90) (layer F.SilkS)
       (effects (font (size 1 1) (thickness 0.15)))
     )
@@
     (descr "28-lead though-hole mounted DIP package, row spacing 15.24 mm (600 mils), Socket")
     (tags "THT DIP DIL PDIP 2.54mm 15.24mm 600mil Socket")
-    (fp_text reference U5 (at 7.62 -2.33 90) (layer F.SilkS)
+    (fp_text reference U5 (at -2.286 1.27 180) (layer F.SilkS)
       (effects (font (size 1 1) (thickness 0.15)))
     )
@@
     (descr "28-lead though-hole mounted DIP package, row spacing 15.24 mm (600 mils)")
     (tags "THT DIP DIL PDIP 2.54mm 15.24mm 600mil")
-    (fp_text reference J1 (at 7.62 -2.33 90) (layer F.SilkS)
+    (fp_text reference J1 (at 7.62 -2.33 90) (layer F.SilkS) hide
       (effects (font (size 1 1) (thickness 0.15)))
     )
@@
     (pad 28 thru_hole oval (at 15.24 0 90) (size 1.6 1.6) (drill 0.8) (layers *.Cu *.Mask)
       (net 23 +9V))
+    (model ${KISYS3DMOD}/Connector_PinHeader_2.54mm.3dshapes/PinHeader_1x14_P2.54mm_Vertical.step
+      (offset (xyz 0 0 -1.75))
+      (scale (xyz 1 1 1))
+      (rotate (xyz 0 180 0))
+    )
+    (model ${KISYS3DMOD}/Connector_PinHeader_2.54mm.3dshapes/PinHeader_1x14_P2.54mm_Vertical.step
+      (offset (xyz 15.24 0 -1.75))
+      (scale (xyz 1 1 1))
+      (rotate (xyz 0 180 0))
+    )
   )
   (module Capacitor_THT:C_Disc_D5.0mm_W2.5mm_P2.50mm (layer F.Cu)
@@
       (effects (font (size 1 1) (thickness 0.15)))
     )
-    (fp_text value CERAMIC (at 1.25 2.5) (layer F.Fab)
+    (fp_text value 100n (at 1.25 2.5) (layer F.Fab)
       (effects (font (size 1 1) (thickness 0.15)))
     )
@@
     (descr "C, Disc series, Radial, pin pitch=2.50mm, , diameter*width=5*2.5mm^2, Capacitor, http://cdn-reichelt.de/documents/datenblatt/B300/DS_KERKO_TC.pdf")
     (tags "C Disc series Radial pin pitch 2.50mm  diameter 5mm width 2.5mm Capacitor")
-    (fp_text reference C1 (at 1.25 -2.5) (layer F.SilkS)
-      (effects (font (size 1 1) (thickness 0.15)))
-    )
-    (fp_text value CERAMIC (at 1.25 2.5) (layer F.Fab)
+    (fp_text reference C1 (at -2.667 -1.397) (layer F.SilkS)
+      (effects (font (size 1 1) (thickness 0.15)))
+    )
+    (fp_text value 100n (at 1.25 2.5) (layer F.Fab)
       (effects (font (size 1 1) (thickness 0.15)))
     )
@@
     (descr "CP, Radial series, Radial, pin pitch=2.50mm, , diameter=6.3mm, Electrolytic Capacitor")
     (tags "CP Radial series Radial pin pitch 2.50mm  diameter 6.3mm Electrolytic Capacitor")
-    (fp_text reference C6 (at -2.834 -0.889 180) (layer F.SilkS)
+    (fp_text reference C6 (at -2.834 -0.635 180) (layer F.SilkS)
       (effects (font (size 1 1) (thickness 0.15)))
     )
@@
     (descr "20-lead though-hole mounted DIP package, row spacing 7.62 mm (300 mils)")
     (tags "THT DIP DIL PDIP 2.54mm 7.62mm 300mil")
-    (fp_text reference U6 (at 3.81 -2.33 90) (layer F.SilkS)
-      (effects (font (size 1 1) (thickness 0.15)))
-    )
-    (fp_text value ADC0804 (at 3.81 25.19 90) (layer F.Fab)
+    (fp_text reference U6 (at 3.81 -2.54 180) (layer F.SilkS)
+      (effects (font (size 1 1) (thickness 0.15)))
+    )
+    (fp_text value ADC0804 (at 3.7325 11.425 180) (layer F.SilkS)
       (effects (font (size 1 1) (thickness 0.15)))
     )
@@
     (descr "Inductor, Axial series, Axial, Horizontal, pin pitch=10.16mm, , length*diameter=6.6*2.7mm^2, Vishay, IM-2, http://www.vishay.com/docs/34030/im.pdf")
     (tags "Inductor Axial series Axial Horizontal pin pitch 10.16mm  length 6.6mm diameter 2.7mm Vishay IM-2")
-    (fp_text reference L1 (at 5.08 -2.47 90) (layer F.SilkS)
-      (effects (font (size 1 1) (thickness 0.15)))
-    )
-    (fp_text value 100 (at 5.08 2.47 90) (layer F.Fab)
+    (fp_text reference L1 (at 2.54 -2.794 180) (layer F.SilkS)
+      (effects (font (size 1 1) (thickness 0.15)))
+    )
+    (fp_text value 100 (at 5.079999 -0.0675 90) (layer F.SilkS)
       (effects (font (size 1 1) (thickness 0.15)))
     )
@@
   (gr_line (start 134.112 100.584) (end 134.112 76.835) (layer Edge.Cuts) (width 0.05))
   (gr_line (start 127 100.584) (end 134.112 100.584) (layer Edge.Cuts) (width 0.05))
-  (gr_text ? (at 167.894 82.042) (layer F.SilkS)
-    (effects (font (size 1 1) (thickness 0.15)))
-  )
   (gr_text ? (at 168.652 84.332) (layer F.SilkS)
     (effects (font (size 1 1) (thickness 0.15)))
   )
-  (gr_text ? (at 150.241 78.867) (layer F.SilkS)
-    (effects (font (size 1 1) (thickness 0.15)))
-  )
-  (gr_text ? (at 135.001 93.853) (layer F.SilkS)
-    (effects (font (size 1 1) (thickness 0.15)))
-  )
-  (gr_text ? (at 143.891 78.359) (layer F.SilkS)
-    (effects (font (size 1 1) (thickness 0.15)))
-  )

Commit message: Fix socket
Parts:
- J1: footprint Package_DIP:DIP-28_W15.24mm -> ReBlast:DIP-28_W15.24mm_Socket
