File: ReBlast.sch (KiCad schematic (older format))
At the start: 21 parts, among them J1 MOS_8580_Socket, U1 74HC20, U2 74LS139, U3 ZN428E-8, U4 TLC272, U5 MOS_8580

Commit message: Checkpoint!
Parts:
- U2: value 74LS139 -> 74HC139
Connections:
- net +5V: now also U1.14 (VCC), U2.16 (VCC)
- net GNDD: now also U1.7 (GND), U2.2 (A0), U2.8 (GND)
- net r_~w: now also U2.14 (A0)
- net a3: now reaches U1.1
- net a3: now also J1.12 (A3), U5.12 (A3)
- net a2: now reaches U1.2
- net a2: now also J1.11 (A2), U5.11 (A2)
- net a1: now reaches U1.4
- net a1: now also J1.10 (A1), U5.10 (A1)
- net a4: now reaches U1.5
- net a4: now also J1.13 (A4), U5.13 (A4)
- net ~digiaddr: now reaches U1.6
- net ~digiaddr: now also U2.3 (A1)
- net ~cs_in: now reaches U2.1 (E)
- net ~cs_in: now also J1.8 (~CS)
- net ~cs_dac_adc: now reaches U2.4 (O0)
- net ~cs_dac_adc: now also U2.15 (E)
- net ~cs_sid: now reaches U2.6 (O2)
- net ~cs_sid: now also U5.8 (~CS)
- net ~cs_adc_w: now reaches U2.10 (O2)
- net ~cs_dac_r: now reaches U2.11 (O1)
- net ~cs_dac_w: now reaches U2.12 (O0)
- net a0: now reaches U2.13 (A1)
- net a0: now also J1.9 (A0), U5.9 (A0)
- net ~cs_adc_r: now reaches U2.9 (O3)
- removed net ~cs: J1.8 (~CS), U5.8 (~CS)
- no-connect marks 1 -> 3
Other:
- note added: "$FD5E"
- note added: "$FD5F"
- note added: "DIGIBLASTER I/O ADDRESS: $fd5e/$fd5f\n(stolen from SID-Card, because unused by SID-Chip)"
- moved on the sheet: U1A, U1B, U2A, U2B, U4A, U4B
Changed lines of the file:
@@
 Sheet 1 1
 Title "ReBlast"
-Date "2022-10-26"
+Date "2022-11-10"
 Rev "1git"
 Comp "SukkoPera"
@@
 L Amplifier_Operational:TLC272 U4
 U 1 1 637D1004
-P 4250 5085
-F 0 "U4" H 4250 5452 50  0000 C CNN
-F 1 "TLC272" H 4250 5361 50  0000 C CNN
-F 2 "Package_DIP:DIP-8_W7.62mm_Socket_LongPads" H 4250 5085 50  0001 C CNN
-F 3 "http://www.ti.com/lit/ds/symlink/tlc272.pdf" H 4250 5085 50  0001 C CNN
-	1    4250 5085
+P 5605 4980
+F 0 "U4" H 5605 5347 50  0000 C CNN
+F 1 "TLC272" H 5605 5256 50  0000 C CNN
+F 2 "Package_DIP:DIP-8_W7.62mm_Socket_LongPads" H 5605 4980 50  0001 C CNN
+F 3 "http://www.ti.com/lit/ds/symlink/tlc272.pdf" H 5605 4980 50  0001 C CNN
+	1    5605 4980
 	1    0    0    -1
 $EndComp
@@
 L Amplifier_Operational:TLC272 U4
 U 2 1 637D42E3
-P 4290 5955
-F 0 "U4" H 4290 6322 50  0000 C CNN
-F 1 "TLC272" H 4290 6231 50  0000 C CNN
-F 2 "Package_DIP:DIP-8_W7.62mm_Socket_LongPads" H 4290 5955 50  0001 C CNN
-F 3 "http://www.ti.com/lit/ds/symlink/tlc272.pdf" H 4290 5955 50  0001 C CNN
-	2    4290 5955
+P 5695 5695
+F 0 "U4" H 5695 6062 50  0000 C CNN
+F 1 "TLC272" H 5695 5971 50  0000 C CNN
+F 2 "Package_DIP:DIP-8_W7.62mm_Socket_LongPads" H 5695 5695 50  0001 C CNN
+F 3 "http://www.ti.com/lit/ds/symlink/tlc272.pdf" H 5695 5695 50  0001 C CNN
+	2    5695 5695
 	1    0    0    -1
 $EndComp
@@
 L 74xx:74LS20 U1
 U 1 1 637E104A
-P 1080 5100
-F 0 "U1" H 1080 5475 50  0000 C CNN
-F 1 "74HC20" H 1080 5384 50  0000 C CNN
-F 2 "Package_DIP:DIP-14_W7.62mm_Socket_LongPads" H 1080 5100 50  0001 C CNN
-F 3 "http://www.ti.com/lit/gpn/sn74LS20" H 1080 5100 50  0001 C CNN
-	1    1080 5100
-	1    0    0    -1
-$EndComp
-$Comp
-L 74xx:74LS20 U1
-U 2 1 637E227B
-P 1095 5780
-F 0 "U1" H 1095 6155 50  0000 C CNN
-F 1 "74HC20" H 1095 6064 50  0000 C CNN
-F 2 "Package_DIP:DIP-14_W7.62mm_Socket_LongPads" H 1095 5780 50  0001 C CNN
-F 3 "http://www.ti.com/lit/gpn/sn74LS20" H 1095 5780 50  0001 C CNN
-	2    1095 5780
+P 1610 3700
+F 0 "U1" H 1610 4075 50  0000 C CNN
+F 1 "74HC20" H 1610 3984 50  0000 C CNN
+F 2 "Package_DIP:DIP-14_W7.62mm_Socket_LongPads" H 1610 3700 50  0001 C CNN
+F 3 "http://www.ti.com/lit/gpn/sn74LS20" H 1610 3700 50  0001 C CNN
+	1    1610 3700
 	1    0    0    -1
 $EndComp
@@
 L 74xx:74LS139 U2
 U 1 1 637E830D
-P 2690 4995
-F 0 "U2" H 2690 5362 50  0000 C CNN
-F 1 "74LS139" H 2690 5271 50  0000 C CNN
-F 2 "Package_DIP:DIP-16_W7.62mm_Socket_LongPads" H 2690 4995 50  0001 C CNN
-F 3 "http://www.ti.com/lit/ds/symlink/sn74ls139a.pdf" H 2690 4995 50  0001 C CNN
-	1    2690 4995
+P 3145 3800
+F 0 "U2" H 3145 4167 50  0000 C CNN
+F 1 "74HC139" H 3145 4076 50  0000 C CNN
+F 2 "Package_DIP:DIP-16_W7.62mm_Socket_LongPads" H 3145 3800 50  0001 C CNN
+F 3 "http://www.ti.com/lit/ds/symlink/sn74ls139a.pdf" H 3145 3800 50  0001 C CNN
+	1    3145 3800
 	1    0    0    -1
 $EndComp
@@
 L 74xx:74LS139 U2
 U 2 1 637E9326
-P 2655 5730
-F 0 "U2" H 2655 6097 50  0000 C CNN
-F 1 "74LS139" H 2655 6006 50  0000 C CNN
-F 2 "Package_DIP:DIP-16_W7.62mm_Socket_LongPads" H 2655 5730 50  0001 C CNN
-F 3 "http://www.ti.com/lit/ds/symlink/sn74ls139a.pdf" H 2655 5730 50  0001 C CNN
-	2    2655 5730
+P 3145 4855
+F 0 "U2" H 3145 5222 50  0000 C CNN
+F 1 "74HC139" H 3145 5131 50  0000 C CNN
+F 2 "Package_DIP:DIP-16_W7.62mm_Socket_LongPads" H 3145 4855 50  0001 C CNN
+F 3 "http://www.ti.com/lit/ds/symlink/sn74ls139a.pdf" H 3145 4855 50  0001 C CNN
+	2    3145 4855
 	1    0    0    -1
 $EndComp
@@
 P 2675 6865
 F 0 "U2" H 2905 6911 50  0000 L CNN
-F 1 "74LS139" H 2905 6820 50  0000 L CNN
+F 1 "74HC139" H 2905 6820 50  0000 L CNN
 F 2 "Package_DIP:DIP-16_W7.62mm_Socket_LongPads" H 2675 6865 50  0001 C CNN
 F 3 "http://www.ti.com/lit/ds/symlink/sn74ls139a.pdf" H 2675 6865 50  0001 C CNN
@@
 r_~w
 Text Label 1130 1995 0    50   ~ 0
-~cs
+~cs_in
 Entry Wire Line
 	1030 2195 1130 2095
@@
 r_~w
 Text Label 4840 1995 0    50   ~ 0
-~cs
+~cs_sid
 Entry Wire Line
 	4740 2195 4840 2095
@@
 Wire Wire Line
 	8465 2540 8465 2130
+Wire Wire Line
+	1310 3550 1170 3550
+Text Label 1170 3550 0    50   ~ 0
+a3
+Text Notes 5065 3635 0    50   ~ 0
+DIGIBLASTER I/O ADDRESS: $fd5e/$fd5f\n(stolen from SID-Card, because unused by SID-Chip)
+Text Label 1130 2095 0    50   ~ 0
+a0
+Text Label 1130 2195 0    50   ~ 0
+a1
+Text Label 1130 2295 0    50   ~ 0
+a2
+Text Label 1130 2395 0    50   ~ 0
+a3
+Text Label 1130 2495 0    50   ~ 0
+a4
+Text Label 4840 2095 0    50   ~ 0
+a0
+Text Label 4840 2195 0    50   ~ 0
+a1
+Text Label 4840 2295 0    50   ~ 0
+a2
+Text Label 4840 2395 0    50   ~ 0
+a3
+Text Label 4840 2495 0    50   ~ 0
+a4
+$Comp
+L 74xx:74LS20 U1
+U 2 1 637E227B
+P 3170 5680
+F 0 "U1" H 3170 6055 50  0000 C CNN
+F 1 "74HC20" H 3170 5964 50  0000 C CNN
+F 2 "Package_DIP:DIP-14_W7.62mm_Socket_LongPads" H 3170 5680 50  0001 C CNN
+F 3 "http://www.ti.com/lit/gpn/sn74LS20" H 3170 5680 50  0001 C CNN
+	2    3170 5680
+	1    0    0    -1
+$EndComp
+$Comp
+L power:+5V #PWR?
+U 1 1 6363E3A4
+P 1150 6270
+F 0 "#PWR?" H 1150 6120 50  0001 C CNN
+F 1 "+5V" H 1165 6443 50  0000 C CNN
+F 2 "" H 1150 6270 50  0001 C CNN
+F 3 "" H 1150 6270 50  0001 C CNN
+	1    1150 6270
+	1    0    0    -1
+$EndComp
+Wire Wire Line
+	1150 6270 1150 6365
+$Comp
+L power:+5V #PWR?
+U 1 1 6364296E
+P 2675 6270
+F 0 "#PWR?" H 2675 6120 50  0001 C CNN
+F 1 "+5V" H 2690 6443 50  0000 C CNN
+F 2 "" H 2675 6270 50  0001 C CNN
+F 3 "" H 2675 6270 50  0001 C CNN
+	1    2675 6270
+	1    0    0    -1
+$EndComp
+Wire Wire Line
+	2675 6270 2675 6365
+Wire Wire Line
+	1150 7365 1150 7460
+$Comp
+L power:GNDD #PWR?
+U 1 1 6364D192
+P 1150 7460
+F 0 "#PWR?" H 1150 7210 50  0001 C CNN
+F 1 "GNDD" H 1154 7305 50  0000 C CNN
+F 2 "" H 1150 7460 50  0001 C CNN
+F 3 "" H 1150 7460 50  0001 C CNN
+	1    1150 7460
+	1    0    0    -1
+$EndComp
+Wire Wire Line
+	2675 7365 2675 7460
+$Comp
+L power:GNDD #PWR?
+U 1 1 6364E268
+P 2675 7460
+F 0 "#PWR?" H 2675 7210 50  0001 C CNN
+F 1 "GNDD" H 2679 7305 50  0000 C CNN
+F 2 "" H 2675 7460 50  0001 C CNN
+F 3 "" H 2675 7460 50  0001 C CNN
+	1    2675 7460
+	1    0    0    -1
+$EndComp
+Wire Wire Line
+	1310 3650 1170 3650
+Wire Wire Line
+	1310 3750 1170 3750
+Wire Wire Line
+	1310 3850 1170 3850
+Text Label 1170 3650 0    50   ~ 0
+a2
+Text Label 1170 3750 0    50   ~ 0
+a1
+Text Label 1170 3850 0    50   ~ 0
+a4
+Wire Wire Line
+	2645 4755 2155 4755
+Text Label 2155 4755 0    50   ~ 0
+a0
+Wire Wire Line
+	3645 4755 4125 4755
+Wire Wire Line
+	3645 3700 4135 3700
+Wire Wire Line
+	3645 3900 4135 3900
+Wire Wire Line
+	2645 4000 2195 4000
+Text Label 2195 4000 0    50   ~ 0
+~cs_in
+Text Notes 4205 4790 0    50   ~ 0
+$FD5E
+Text Notes 4205 4990 0    50   ~ 0
+$FD5F
+Text Label 4125 4755 2    50   ~ 0
+~cs_dac_w
+Wire Wire Line
+	1910 3700 2645 3700
+Text Label 2080 3700 0    50   ~ 0
+~digiaddr
+Wire Wire Line
+	2645 4855 2155 4855
+Text Label 2155 4855 0    50   ~ 0
+r_~w
+Wire Wire Line
+	2645 3800 2555 3800
+Wire Wire Line
+	2555 3800 2555 4140
+$Comp
+L power:GNDD #PWR?
+U 1 1 636EFB85
+P 2555 4140
+F 0 "#PWR?" H 2555 3890 50  0001 C CNN
+F 1 "GNDD" H 2559 3985 50  0000 C CNN
+F 2 "" H 2555 4140 50  0001 C CNN
+F 3 "" H 2555 4140 50  0001 C CNN
+	1    2555 4140
+	1    0    0    -1
+$EndComp
+Text Label 4135 3700 2    50   ~ 0
+~cs_dac_adc
+Text Label 4135 3900 2    50   ~ 0
+~cs_sid
+NoConn ~ 3645 3800
+NoConn ~ 3645 4000
+Wire Wire Line
+	2645 5055 2155 5055
+Text Label 2155 5055 0    50   ~ 0
+~cs_dac_adc
+Wire Wire Line
+	3645 4855 4125 4855
+Text Label 4125 4855 2    50   ~ 0
+~cs_dac_r
+Wire Wire Line
+	3645 4955 4125 4955
+Text Label 4125 4955 2    50   ~ 0
+~cs_adc_w
+Wire Wire Line
+	3645 5055 4125 5055
+Text Label 4125 5055 2    50   ~ 0
+~cs_adc_r
 Wire Bus Line
 	8465 940  8465 1430
 Wire Bus Line
+	4740 2195 4740 2595
+Wire Bus Line
 	1030 2195 1030 2595
 Wire Bus Line
-	4740 2195 4740 2595
-Wire Bus Line
 	10465 940  10465 1830

Commit message: Suppositions in progress...
Parts:
- added C7: 6.8u, Capacitor_THT:CP_Radial_D5.0mm_P2.00mm, symbol Device:CP1
- added U6: ZN427E8, MODULE, symbol ZN427E8:ZN427E8
- C2: footprint Capacitor_THT:CP_Radial_D5.0mm_P2.00mm -> Capacitor_THT:C_Disc_D7.0mm_W2.5mm_P5.00mm
- C3: value 1u -> 4.7u
- C4: value CP1 -> 680n
- D1: value 1n4148 -> 2.5V ZENER
- R2: value 4.7k -> 47k
- R4: value 10K or 120 -> 10K
Connections:
- net +5V: now also U1.10, U1.12, U1.9, U6.10 (VCC)
- net GNDA: no longer C3.2
- net GNDD: now also C3.2, D1.2 (A), D3.1 (K), C7.2, U6.9 (GND)
- net audio_in: now also R4.2, U4.7
- net d0: now also U6.11 (BIT1)
- net d1: now also U6.12 (BIT2)
- net d2: now also U6.13 (BIT3)
- net d3: now also U6.14 (BIT4)
- net d4: now also U6.15 (BIT5)
- net d5: now also U6.16 (BIT6)
- net d6: now also U6.17 (BIT7)
- net d7: now also U6.18 (BIT8)
- net phi2: now also C4.1, U6.3 (CLOCK)
- net ~cs_adc_r: now also U1.13; no longer U2.9 (O3)
- net ~cs_adc_w: now also U6.4 (~WR)
- net ~cs_dac_w: now also U3.4 (ENABLE)
- net dac_output: now reaches U4.5 (+)
- net dac_output: now also U3.5 (AOUT)
- net at U4.6 (-): now also R4.1
- net vref: now reaches C3.1, R5.2, U3.6 (VREF_IN), U3.7 (VREF_OUT)
- net vref: now also D1.1 (K), U6.7 (VREF_IN), U6.8 (VREF_OUT)
- net at R2.1: now also U6.5 (REXT)
- net at R2.2: now also D2.2 (A), C7.1
- net at D2.1 (K): now also C4.2, D3.2 (A)
- net audio_jack: now reaches J1.26 (AUDIO_IN)
- net audio_jack: now also U6.6 (VIN)
- new net cs_adc_r: U6.2 (RD)
- no-connect marks 3 -> 8
Other:
- note added: "ADDRESS DECODING"
- note added: "ANALOG-TO-DIGITAL\nCONVERTER"
- note added: "DIGITAL-TO-ANALOG-\nCONVERTER"
- note added: "Maybe decoupling\nfor opamp?"
- note added: "Maybe not\nelectrolytic?"
- note added: "Maybe only one of the 427 or\n428 VREF_OUT should be\nconnected?"
- note added: "Note we must NOT enable SID for\nthe addresses we "steal"!"
- note added: "Or inductor?"
- note added: "Rext, should\nbe 56k, also\nunsure whether\nlast ring is\nbrown/red/orange...\n"
- note added: "SPARES"
- note added: "Simplified version of "Diode Pump" circuit\nfrom ZN427 datasheet: produces a negative\nvoltage sufficient for operation of that IC."
- note added: "There is probably a typo in the ZN427 datasheet:\nthe RD signal is first indicated as "~RD~", which\nwould imply it is active-low, but a timing diagram\na few pages later shows it as a positive pulse, and\nit is also indicated again as "RD" further on."
- note added: "VREF GENERATION CIRCUIT\n(From datasheets)"
- note added: "We'd need a 20k\nresistor here..."
- note added: "ZN427 datasheet says 1u\nZN428 datasheet says 4.7u\nThe latter should be fine for both.\nDatasheets say this circuit can\ndrive up to 5 ICs so it should be\nfine for just 2."
- moved on the sheet: C1, C2, C3, C4, C5, C6, D1, D2, D3, J1, R1, R2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

Commit message: Back side is 99% done. Top side is full of doubts...
Parts:
- removed U6: ZN427E8, MODULE, symbol ZN427E8:ZN427E8
- added U6: ADC0804, Package_DIP:DIP-20_W7.62mm, symbol ADC0804:ADC0804
- C1: footprint Capacitor_THT:C_Disc_D7.0mm_W2.5mm_P5.00mm -> Capacitor_THT:C_Disc_D5.0mm_W2.5mm_P2.50mm
- C2: value C_TANTALUM -> 4.7u; footprint Capacitor_THT:C_Disc_D7.0mm_W2.5mm_P5.00mm -> Capacitor_THT:C_Disc_D5.0mm_W2.5mm_P2.50mm
- C3: value 4.7u -> 1u
- C4: value 680n -> C
- C6: footprint Capacitor_THT:CP_Radial_D8.0mm_P5.00mm -> Capacitor_THT:CP_Radial_D6.3mm_P2.50mm
- J1: footprint ReBlast:DIP-28_Socket_LongPads -> Package_DIP:DIP-28_W15.24mm
- R2: value 47k -> 4.7k
- R3: footprint Resistor_THT:R_Axial_DIN0414_L11.9mm_D4.5mm_P15.24mm_Horizontal -> Resistor_THT:R_Axial_DIN0207_L6.3mm_D2.5mm_P7.62mm_Horizontal
- U3: footprint Package_DIP:DIP-16_W7.62mm_Socket_LongPads -> Package_DIP:DIP-16_W7.62mm_Socket
- U4: footprint Package_DIP:DIP-8_W7.62mm_Socket_LongPads -> Package_DIP:DIP-8_W7.62mm_Socket
- U5: footprint Package_DIP:DIP-28_W15.24mm_Socket_LongPads -> Package_DIP:DIP-28_W15.24mm_Socket
Connections:
- net labels added: ~cs_adc, ~cs_dac
- net labels removed: cs_adc_r, ~cs_adc_w, ~cs_dac_r, ~cs_dac_w
- wire segments 164 -> 178
- no-connect marks 8 -> 5
Other:
- note added: "100k ON\nSOME BOARDS"
- note added: "CHIP D1 = MSB\nVERY CONFUSING\nNUMBERING!"
- note added: "Tantalum\ngoes here?"
- note removed: "Maybe decoupling\nfor opamp?"
- note removed: "Maybe not\nelectrolytic?"
- note removed: "Maybe only one of the 427 or\n428 VREF_OUT should be\nconnected?"
- note removed: "Rext, should\nbe 56k, also\nunsure whether\nlast ring is\nbrown/red/orange...\n"
- note removed: "SPARES"
- note removed: "Simplified version of "Diode Pump" circuit\nfrom ZN427 datasheet: produces a negative\nvoltage sufficient for operation of that IC."
- note removed: "There is probably a typo in the ZN427 datasheet:\nthe RD signal is first indicated as "~RD~", which\nwould imply it is active-low, but a timing diagram\na few pages later shows it as a positive pulse, and\nit is also indicated again as "RD" further on."
- note removed: "We'd need a 20k\nresistor here..."
- note removed: "ZN427 datasheet says 1u\nZN428 datasheet says 4.7u\nThe latter should be fine for both.\nDatasheets say this circuit can\ndrive up to 5 ICs so it should be\nfine for just 2."
- moved on the sheet: C1, C2, C3, C4, C5, C6, C7, D1, D2, D3, R1, R2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

Commit message: Power circuit almost makes sense
Parts:
- removed R3: 100R 1/2W, Resistor_THT:R_Axial_DIN0207_L6.3mm_D2.5mm_P7.62mm_Horizontal, symbol Device:R
- added L1: 100, Inductor_THT:L_Axial_L6.6mm_D2.7mm_P10.16mm_Horizontal_Vishay_IM-2, symbol Device:L
Connections:
- net labels added: VCC
Other:
- note added: "INPUT\nPOWER\nFILTER"
- note removed: "Or inductor?"
- moved on the sheet: C6
Changed lines of the file:
@@
 	3730 2110 3730 1485
-$Comp
-L power:+5V #PWR0105
-U 1 1 638225B0
-P 3730 1485
-F 0 "#PWR0105" H 3730 1335 50  0001 C CNN
-F 1 "+5V" H 3850 1520 50  0000 C CNN
-F 2 "" H 3730 1485 50  0001 C CNN
-F 3 "" H 3730 1485 50  0001 C CNN
-	1    3730 1485
-	1    0    0    -1
-$EndComp
 $Comp
 L power:+9V #PWR0106
@@
 	7490 2110 7490 1485
 $Comp
-L power:+5V #PWR0108
-U 1 1 6388753C
-P 7490 1485
-F 0 "#PWR0108" H 7490 1335 50  0001 C CNN
-F 1 "+5V" H 7505 1658 50  0000 C CNN
-F 2 "" H 7490 1485 50  0001 C CNN
-F 3 "" H 7490 1485 50  0001 C CNN
-	1    7490 1485
-	1    0    0    -1
-$EndComp
-$Comp
 L power:+9V #PWR0109
 U 1 1 63887546
@@
 Wire Wire Line
 	6360 6905 5875 6905
-Wire Wire Line
-	8270 9500 7930 9500
-Connection ~ 8270 9500
-Wire Wire Line
-	8270 9625 8270 9500
-Wire Wire Line
-	8630 9500 8270 9500
-Text Notes 8540 9645 0    50   ~ 0
-Or inductor?
+Connection ~ 4450 9685
+Wire Wire Line
+	4450 9810 4450 9685
+Wire Wire Line
+	4255 9685 4450 9685
 $Comp
 L Device:C C1
@@
 L Device:CP1 C6
 U 1 1 637F2B75
-P 8270 9775
-F 0 "C6" H 8385 9821 50  0000 L CNN
-F 1 "CP1" H 8385 9730 50  0000 L CNN
-F 2 "Capacitor_THT:CP_Radial_D6.3mm_P2.50mm" H 8270 9775 50  0001 C CNN
-F 3 "~" H 8270 9775 50  0001 C CNN
-	1    8270 9775
-	1    0    0    -1
-$EndComp
-$Comp
-L Device:R R3
-U 1 1 637EE040
-P 8780 9500
-F 0 "R3" V 8987 9500 50  0000 C CNN
-F 1 "100R 1/2W" V 8896 9500 50  0000 C CNN
-F 2 "Resistor_THT:R_Axial_DIN0207_L6.3mm_D2.5mm_P7.62mm_Horizontal" V 8710 9500 50  0001 C CNN
-F 3 "~" H 8780 9500 50  0001 C CNN
-	1    8780 9500
-	0    -1   -1   0
+P 4450 9960
+F 0 "C6" H 4565 10006 50  0000 L CNN
+F 1 "CP1" H 4565 9915 50  0000 L CNN
+F 2 "Capacitor_THT:CP_Radial_D6.3mm_P2.50mm" H 4450 9960 50  0001 C CNN
+F 3 "~" H 4450 9960 50  0001 C CNN
+	1    4450 9960
+	-1   0    0    -1
 $EndComp
 $Comp
@@
 	0    1    1    0
 $EndComp
-Connection ~ 7930 9500
 Wire Wire Line
 	7930 9500 7400 9500
@@
 	8815 7005 8930 7005
 Wire Wire Line
-	6660 6905 6765 6905
-Wire Wire Line
 	5905 9590 5905 9500
 Wire Wire Line
@@
 Wire Wire Line
 	7355 6905 7625 6905
-Wire Wire Line
-	6910 6695 6765 6695
-Wire Wire Line
-	6765 6695 6765 6905
-Connection ~ 6765 6905
-Wire Wire Line
-	6765 6905 6900 6905
 NoConn ~ 12605 7985
 Wire Wire Line
@@
 L power:GNDA #PWR0116
 U 1 1 6490D101
-P 8270 10040
-F 0 "#PWR0116" H 8270 9790 50  0001 C CNN
-F 1 "GNDA" H 8275 9867 50  0000 C CNN
-F 2 "" H 8270 10040 50  0001 C CNN
-F 3 "" H 8270 10040 50  0001 C CNN
-	1    8270 10040
-	1    0    0    -1
-$EndComp
-Wire Wire Line
-	8270 9925 8270 10040
+P 4450 10225
+F 0 "#PWR0116" H 4450 9975 50  0001 C CNN
+F 1 "GNDA" H 4455 10052 50  0000 C CNN
+F 2 "" H 4450 10225 50  0001 C CNN
+F 3 "" H 4450 10225 50  0001 C CNN
+	1    4450 10225
+	-1   0    0    -1
+$EndComp
+Wire Wire Line
+	4450 10110 4450 10225
 $Comp
 L Device:R R4
@@
 Wire Wire Line
 	6730 10000 6925 10000
+Wire Wire Line
+	6660 6905 6900 6905
+Wire Wire Line
+	4450 9685 4450 9575
+$Comp
+L power:+5V #PWR0121
+U 1 1 65EB97C5
+P 4450 9575
+F 0 "#PWR0121" H 4450 9425 50  0001 C CNN
+F 1 "+5V" H 4465 9748 50  0000 C CNN
+F 2 "" H 4450 9575 50  0001 C CNN
+F 3 "" H 4450 9575 50  0001 C CNN
+	1    4450 9575
+	-1   0    0    -1
+$EndComp
+Wire Wire Line
+	3955 9685 3760 9685
+Wire Wire Line
+	3760 9685 3760 9575
+$Comp
+L Device:L L1
+U 1 1 65ED0D04
+P 4105 9685
+F 0 "L1" V 3924 9685 50  0000 C CNN
+F 1 "100" V 4015 9685 50  0000 C CNN
+F 2 "Inductor_THT:L_Axial_L6.6mm_D2.7mm_P10.16mm_Horizontal_Vishay_IM-2" H 4105 9685 50  0001 C CNN
+F 3 "~" H 4105 9685 50  0001 C CNN
+	1    4105 9685
+	0    -1   1    0
+$EndComp
+$Comp
+L power:VCC #PWR01
+U 1 1 65EDD900
+P 3760 9575
+F 0 "#PWR01" H 3760 9425 50  0001 C CNN
+F 1 "VCC" H 3775 9748 50  0000 C CNN
+F 2 "" H 3760 9575 50  0001 C CNN
+F 3 "" H 3760 9575 50  0001 C CNN
+	1    3760 9575
+	-1   0    0    -1
+$EndComp
+Text Notes 3985 9190 0    50   ~ 0
+INPUT\nPOWER\nFILTER
+Wire Wire Line
+	7930 9035 7930 8925
+$Comp
+L power:+5V #PWR0126
+U 1 1 65F29FC9
+P 7930 8925
+F 0 "#PWR0126" H 7930 8775 50  0001 C CNN
+F 1 "+5V" H 7945 9098 50  0000 C CNN
+F 2 "" H 7930 8925 50  0001 C CNN
+F 3 "" H 7930 8925 50  0001 C CNN
+	1    7930 8925
+	-1   0    0    -1
+$EndComp
+Connection ~ 7930 9035
 Wire Bus Line
 	12335 4055 12335 4545
@@
 Wire Bus Line
 	14355 7285 14355 8385
+$Comp
+L power:VCC #PWR?
+U 1 1 65F3A32A
+P 3730 1485
+F 0 "#PWR?" H 3730 1335 50  0001 C CNN
+F 1 "VCC" H 3745 1658 50  0000 C CNN
+F 2 "" H 3730 1485 50  0001 C CNN
+F 3 "" H 3730 1485 50  0001 C CNN
+	1    3730 1485
+	-1   0    0    -1
+$EndComp
+$Comp
+L power:VCC #PWR?
+U 1 1 65F3BEFA
+P 7490 1485
+F 0 "#PWR?" H 7490 1335 50  0001 C CNN
+F 1 "VCC" H 7432 1522 50  0000 R CNN
+F 2 "" H 7490 1485 50  0001 C CNN
+F 3 "" H 7490 1485 50  0001 C CNN
+	1    7490 1485
+	-1   0    0    -1
+$EndComp
 $EndSCHEMATC

Commit message: Nothing makes sense
Parts:
- removed C2: 4.7u, Capacitor_THT:C_Disc_D5.0mm_W2.5mm_P2.50mm, symbol Device:CP1
- removed D2, D3: 1N5817, Diode_THT:D_DO-41_SOD81_P2.54mm_Vertical_AnodeUp, symbol Diode:1N5817
- added C2: CERAMIC, Capacitor_THT:C_Disc_D5.0mm_W2.5mm_P2.50mm, symbol Device:C
- added R3, R6: R, Resistor_THT:R_Axial_DIN0207_L6.3mm_D2.5mm_P2.54mm_Vertical, symbol Device:R
- C4: value C -> 1u
- C6: value CP1 -> 47u
- C7: value 6.8u -> 1u
Connections:
- wire segments 178 -> 180
Other:
- note added: "DOESN'T MAKE MUCH SENSE TO ME..."
- note added: "NOT SURE"
- note added: "PROBABLY MORE\nTHAN 1u ON ACTUAL\nCARD"
- note added: "PROPER DIGITAL/ANALOG\nGROUND SEPARATION TBD"
- note removed: "Tantalum\ngoes here?"
- moved on the sheet: R1, R2, RV1

Commit message: Done?
Parts:
- C3: value 1u -> 4.7u
- R3, R6: value R -> 330k
- R4: value 10K -> 100k
Connections:
- net +5V: now also R2.1; no longer U1.10, U1.12, U1.13, U1.14 (VCC), U2.16 (VCC)
- net GNDA: now also U6.7 (VIN-), U6.8 (AGND); no longer R3.2
- net VCC: now also U1.10, U1.12, U1.13, U1.14 (VCC), U2.16 (VCC)
- net phi2: now also U6.4 (CLK_IN)
- net r_~w: now also U1.9
- net adc_vref_half: now reaches R6.1, U4.1
- net adc_vref_half: now also U6.9 (VREF_HALF)
- net at U4.3 (+): now also RV1.2
- net at C7.1, U4.5 (+): now also C2.1, D1.2 (A), R2.2
- net adc_in: now reaches U4.7
- net adc_in: now also R3.2, U6.6 (VIN+)
- net ~read: now reaches U1.8
- net ~read: now also U6.2 (~RD)
- net at R1.2, RV1.1: no longer R2.1
- no-connect marks 5 -> 7
Other:
- note added: "10k ON\nSOME BOARDS"
- note added: "1u ON DATASHEET"
- note added: "NO CAP HERE? :(\nAND R6 DOESN'T MAKE MUCH SENSE..."
- note added: "TOO BAD THIS ZENER\nDIODE IS BACKWARDS..."
- note removed: "100k ON\nSOME BOARDS"
- note removed: "DOESN'T MAKE MUCH SENSE TO ME..."
- note removed: "PROBABLY MORE\nTHAN 1u ON ACTUAL\nCARD"
- moved on the sheet: C1, C2, C5, C7, D1, R1, R2, R3, R4, R6, RV1, U1B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

Commit message: Try to come up with some values for caps
Parts:
- C1, C2: value CERAMIC -> 100n
Other:
- note added: "APPARENTLY R6 DOESN'T MAKE MUCH SENSE,\nBUT IT MIGHT BE THERE TO COMPENSATE FOR\nTHE INPUT IMPEDENCE?"
- note added: "FULL SCALE ADJUSTMENT"
- note added: "INPUT AMPLIFIER\n(Gain = 3.3x)"
- note added: "Note we must NOT enable SID for\nthe addresses we "steal"!\n(Thanks TLC)"
- note added: "TODO: Add 100nF caps for U1/U2"
- note added: "Works as a simple inverter"
- note added: "~cs_in~ is asserted for $FD40-$FD5F\n(and $FE80-$FE9F)"
- note removed: "NO CAP HERE? :(\nAND R6 DOESN'T MAKE MUCH SENSE..."
- note removed: "NOT SURE"
- note removed: "Note we must NOT enable SID for\nthe addresses we "steal"!"
- moved on the sheet: C1, C6, L1, R1, R6, RV1, U1B, U4A

Commit message: Fix socket
Parts:
- J1: footprint Package_DIP:DIP-28_W15.24mm -> ReBlast:DIP-28_W15.24mm_Socket
Changed lines of the file:
@@
 F 0 "J1" H 2800 3475 50  0000 C CNN
 F 1 "MOS_8580_Socket" H 2800 3384 50  0000 C CNN
-F 2 "Package_DIP:DIP-28_W15.24mm" H 2800 2460 50  0001 C CNN
+F 2 "ReBlast:DIP-28_W15.24mm_Socket" H 2800 2460 50  0001 C CNN
 F 3 "DOCUMENTATION" H 2800 2460 50  0001 C CNN
 	1    2800 2460
